Commit message: created_desk_walking_robot in xacro format This includes use of variables

File: ros2_ws/src/desk_walking_robot_description/urdf/my_robot.urdf (robot description, URDF)
Before this commit: robot desktop_crawler, 6 links, 5 joints
Links:
- added link left_ankle_link; visual cylinder length=0.25 radius=0.2
- added link left_foot_link; visual box size=0.5 0.35 0.3
- added link right_ankle_link; visual cylinder length=0.25 radius=0.2
- added link right_foot_link; visual box size=0.5 0.35 0.3
Joints:
- added joint left_ankle_joint: type continuous, parent left_leg_link, child left_ankle_link, origin xyz=0 0 -0.5 rpy=0 0 0, axis 0 -1 0
- added joint left_foot_joint: type fixed, parent left_ankle_link, child left_foot_link, origin xyz=0 0 -0.2 rpy=0 0 0
- added joint right_ankle_joint: type continuous, parent right_leg_link, child right_ankle_link, origin xyz=0 0 -0.5 rpy=0 0 0, axis 0 1 0
- added joint right_foot_joint: type fixed, parent right_ankle_link, child right_foot_link, origin xyz=0 0 -0.2 rpy=0 0 0
- joint base_joint: origin xyz=0 0 0.65 rpy=0 0 0 -> xyz=0 0 0.95 rpy=0 0 0
- joint left_hip_joint: axis 0 1 0 -> -1 0 0
- joint left_leg_joint: origin xyz=0 0 -0.15 rpy=0 0 0 -> xyz=0 0 -0.2 rpy=0 0 0
- joint right_hip_joint: axis 0 -1 0 -> -1 0 0
- joint right_leg_joint: origin xyz=0 0 -0.15 rpy=0 0 0 -> xyz=0 0 -0.2 rpy=0 0 0
