Commit message: desk_walking_robot: add collision and inertia to URDF

File: ros2_ws/src/desk_walking_robot_description/urdf/common_properties.xacro (robot description, xacro)
@@ -11,7 +11,7 @@
             <origin xyz="${xyz}" rpy="${rpy}" />
             <mass value="${mass}" />
-            <inertia ixx="${(mass/12) * (height*height + lenght*lenght)}" ixy="0" ixz="0"
-                     iyy="${(mass/12) * (width*width + lenght*lenght)}" iyz="0"
-                     izz="${(mass/12) * (width*width + height*height)}" />
+            <inertia ixx="${(mass/12) * (width*width + height*height)}" ixy="0" ixz="0"
+                     iyy="${(mass/12) * (lenght*lenght + height*height)}" iyz="0"
+                     izz="${(mass/12) * (lenght*lenght + width*width)}" />
         </inertial>
     </xacro:macro>

File: ros2_ws/src/desk_walking_robot_description/urdf/solid_structure.xacro (robot description, xacro)
@@ -4,10 +4,12 @@
     <xacro:property name="torso_length" value="${0.7 * torso_height}" />
     <xacro:property name="torso_width" value="${0.5 * torso_height}" />
-    <xacro:property name="pivot_radius" value="${0.15 * torso_height}" />
+    <xacro:property name="pivot_radius" value="${0.05 * torso_height}" />
+	<xacro:property name="pivot_length" value="${torso_width/8}" />
     <xacro:property name="leg_lenght" value="${torso_height / 2}" />
-    <xacro:property name="leg_hip_offset" value="${-(leg_lenght / 2) + (pivot_radius * 0.25)}" />
+    <xacro:property name="leg_hip_offset" value="${-(leg_lenght / 2)}" />
     <xacro:property name="leg_ankle_offset" value="${-leg_lenght-pivot_radius*0.5}" />
     <xacro:property name="foot_height" value="${pivot_radius*1.25}" />
     <xacro:property name="foot_ankle_offset" value="${pivot_radius-(foot_height/2)}" />
+	<!-- for wheels collisions use spheres instead of cylinders -->
     <link name="base_footprint" />
     <link name="base_link">
@@ -19,20 +21,28 @@
             <material name="blue" />
         </visual>
+		<collision>
+            <geometry>
+                <box size="${torso_length} ${torso_width} ${torso_height}" />
+            </geometry>
+            <origin xyz="0 0 ${torso_height / 2.0}" rpy="0 0 0" />
+        </collision>
+		<xacro:box_inertia mass="5.0" height="${torso_height}" lenght="${torso_length}" width="${torso_width}"
+                           xyz="0 0 ${torso_height / 2.0}" rpy="0 0 0" />
     </link>
-    <xacro:macro name="pivot_link" params="prefix rpy">
+    <xacro:macro name="pivot_link" params="prefix xyz rpy">
         <link name="${prefix}_link">
             <visual>
                 <geometry>
-                    <cylinder radius="${pivot_radius}" length="${torso_width/4}" />
+                    <cylinder radius="${pivot_radius}" length="${pivot_length}" />
                 </geometry>
-                <origin xyz="0 0 0" rpy="${rpy}" />
+                <origin xyz="${xyz}" rpy="${rpy}" />
                 <material name="grey" />
             </visual>
         </link>
     </xacro:macro>
-    <xacro:pivot_link prefix="right_hip" rpy="0 ${pi/2.0} 0" />
-    <xacro:pivot_link prefix="left_hip" rpy="0 ${pi/2.0} 0" />
-    <xacro:pivot_link prefix="right_ankle" rpy="${pi/2.0} 0 0" />
-    <xacro:pivot_link prefix="left_ankle" rpy="${pi/2.0} 0 0" />
+    <xacro:pivot_link prefix="right_hip" xyz="0 0 -${pivot_length/2}" rpy="0 0 0" />
+    <xacro:pivot_link prefix="left_hip" xyz="0 0 -${pivot_length/2}" rpy="0 0 0" />
+    <xacro:pivot_link prefix="right_ankle" xyz="0 0 0" rpy="${pi/2.0} 0 0" />
+    <xacro:pivot_link prefix="left_ankle" xyz="0 0 0" rpy="${pi/2.0} 0 0" />
     <link name="right_leg_link">
         <visual>
@@ -43,4 +53,11 @@
             <material name="blue" />
         </visual>
+		<collision>
+            <geometry>
+                <cylinder radius="${torso_length*0.2}" length="${leg_lenght}" />
+            </geometry>
+            <origin xyz="0 0 ${leg_hip_offset}" rpy="0 0 0" />
+        </collision>
+		<xacro:cylinder_inertia mass="2.0" radius="${torso_length*0.2}" height="${leg_lenght}" xyz="0 0 ${leg_hip_offset}" rpy="0 0 0" />
     </link>
     <link name="left_leg_link">
@@ -52,4 +69,11 @@
             <material name="blue" />
         </visual>
+		<collision>
+            <geometry>
+                <cylinder radius="${torso_length*0.2}" length="${leg_lenght}" />
+            </geometry>
+            <origin xyz="0 0 ${leg_hip_offset}" rpy="0 0 0" />
+        </collision>
+		<xacro:cylinder_inertia mass="2.0" radius="${torso_length*0.2}" height="${leg_lenght}" xyz="0 0 ${leg_hip_offset}" rpy="0 0 0" />
     </link>
     <link name="right_foot_link">
@@ -61,4 +85,12 @@
             <material name="blue" />
         </visual>
+		<collision>
+            <geometry>
+                <box size="${torso_length*0.5/0.7} ${torso_width*1.1} ${foot_height}" />
+            </geometry>
+            <origin xyz="0 0 ${foot_ankle_offset}" rpy="0 0 0" />
+        </collision>
+		<xacro:box_inertia mass="1.0" lenght="${torso_length*0.5/0.7}" width="${torso_width*1.1}" height="${foot_height}"
+                           xyz="0 0 ${foot_ankle_offset}" rpy="0 0 0" />
     </link>
     <link name="left_foot_link">
@@ -70,4 +102,12 @@
             <material name="blue" />
         </visual>
+		<collision>
+            <geometry>
+                <box size="${torso_length*0.5/0.7} ${torso_width*1.1} ${foot_height}" />
+            </geometry>
+            <origin xyz="0 0 ${foot_ankle_offset}" rpy="0 0 0" />
+        </collision>
+		<xacro:box_inertia mass="1.0" lenght="${torso_length*0.5/0.7}" width="${torso_width*1.1}" height="${foot_height}"
+                           xyz="0 0 ${foot_ankle_offset}" rpy="0 0 0" />
     </link>
     <joint name="base_joint" type="fixed">
@@ -80,5 +120,5 @@
         <child link="right_hip_link" />
         <origin xyz="${torso_length/2} 0 0" rpy="0 0 0"/>
-        <axis xyz="-1 0 0" />
+        <axis xyz="0 0 1" />
         <limit lower="${-pi/2.0}" upper="${pi/2.0}" velocity="100" effort="100" />
     </joint>
@@ -87,5 +127,5 @@
         <child link="left_hip_link" />
         <origin xyz="${-torso_length/2} 0 0" rpy="0 0 0"/>
-        <axis xyz="-1 0 0" />
+        <axis xyz="0 0 -1" />
         <limit lower="${-pi/2.0}" upper="${pi/2.0}" velocity="100" effort="100" />
     </joint>
@@ -93,10 +133,10 @@
         <parent link="right_hip_link" />
         <child link="right_leg_link" />
-        <origin xyz="0 0 -${pivot_radius}" rpy="0 0 0"/>
+        <origin xyz="0 0 -${pivot_length}" rpy="0 0 0"/>
     </joint>
     <joint name="left_leg_joint" type="fixed">
         <parent link="left_hip_link" />
         <child link="left_leg_link" />
-        <origin xyz="0 0 -${pivot_radius}" rpy="0 0 0"/>
+        <origin xyz="0 0 -${pivot_length}" rpy="0 0 0"/>
     </joint>
     <joint name="right_ankle_joint" type="revolute">
