Commit message: desk robot - add camera

File: ros2_ws/src/desk_walking_robot_description/urdf/my_robot.urdf.xacro (robot description, xacro)
@@ -6,3 +6,4 @@
     <!-- Comment  below line if using non-gazebo-plugins version -->
     <xacro:include filename="solid_structure_gazebo.xacro" />
+    <xacro:include filename="camera.xacro" />
 </robot>

File: ros2_ws/src/desk_walking_robot_description/urdf/solid_structure.xacro (robot description, xacro)
@@ -14,5 +14,5 @@
 	<!-- for wheels collisions use spheres instead of cylinders -->
     <link name="base_footprint" />
-    <link name="base_link">
+    <link name="torso_link">
         <visual>
             <geometry>
@@ -114,9 +114,9 @@
     <joint name="base_joint" type="fixed">
         <parent link="base_footprint" />
-        <child link="base_link" />
+        <child link="torso_link" />
         <origin xyz="0 0 ${leg_lenght+foot_height+1.5*pivot_radius}" rpy="0 0 0"/>
     </joint>
     <joint name="right_hip_joint" type="revolute">
-        <parent link="base_link" />
+        <parent link="torso_link" />
         <child link="right_hip_link" />
         <origin xyz="${torso_length/2} 0 0" rpy="0 0 0"/>
@@ -125,5 +125,5 @@
     </joint>
     <joint name="left_hip_joint" type="revolute">
-        <parent link="base_link" />
+        <parent link="torso_link" />
         <child link="left_hip_link" />
         <origin xyz="${-torso_length/2} 0 0" rpy="0 0 0"/>
