Commit message: desk robot - add camera

File: ros2_ws/src/desk_walking_robot_description/urdf/camera.xacro (robot description, xacro)
@@ -17,5 +17,5 @@
             </geometry>
         </collision>
-        <xacro:box_inertia mass="1.0" lenght="${camera_length}" width="${camera_width}" height="${camera_height}"
+        <xacro:box_inertia mass="0.1" lenght="${camera_length}" width="${camera_width}" height="${camera_height}"
                            xyz="0 0 0" rpy="0 0 0" />
     </link>
@@ -23,5 +23,5 @@
         <parent link="torso_link"/>
         <child link="camera_link"/>
-        <origin xyz="0 ${torso_width / 2} ${torso_height / 2}" rpy="0 0 ${pi/2}"/>
+        <origin xyz="0 ${(torso_width + camera_length) / 2} ${torso_height / 2}" rpy="0 0 ${pi/2}"/>
     </joint>
 </robot>

Commit message: enable camera to desk_robot

File: ros2_ws/src/desk_walking_robot_description/urdf/camera.xacro (robot description, xacro)
@@ -25,3 +25,36 @@
         <origin xyz="0 ${(torso_width + camera_length) / 2} ${torso_height / 2}" rpy="0 0 ${pi/2}"/>
     </joint>
+    <link name="camera_link_optical" />
+    <joint name="camera_optical_joint" type="fixed">
+        <origin xyz="0 0 0" rpy="${-pi/2} 0 ${-pi/2}"/>
+        <parent link="camera_link"/>
+        <child link="camera_link_optical"/>
+    </joint>
+    <gazebo reference="camera_link">
+        <sensor name="camera" type="camera">
+            <camera>
+                <horizontal_fov>1.3962634</horizontal_fov>
+                <image>
+                    <width>640</width>
+                    <height>480</height>
+                    <format>R8G8B8</format>
+                </image>
+                <clip>
+                    <near>0.1</near>
+                    <far>15</far>
+                </clip>
+                <noise>
+                    <type>gaussian</type>
+                    <mean>0.0</mean>
+                    <stddev>0.007</stddev>
+                </noise>
+                <optical_frame_id>camera_link_optical</optical_frame_id>
+                <camera_info_topic>camera/camera_info</camera_info_topic>
+            </camera>
+            <always_on>1</always_on>
+            <update_rate>20</update_rate>
+            <visualize>true</visualize>
+            <topic>camera/image_raw</topic>
+        </sensor>
+    </gazebo>
 </robot>

Commit message: format to desk robot files

File: ros2_ws/src/desk_walking_robot_description/urdf/camera.xacro (robot description, xacro)
@@ -7,27 +7,28 @@
         <visual>
             <geometry>
-                <box size="${camera_length} ${camera_width} ${camera_height}"/>
+                <box size="${camera_length} ${camera_width} ${camera_height}" />
             </geometry>
-            <material name="grey"/>
+            <material name="grey" />
             <!-- origin is 0 0 0 -->
         </visual>
         <collision>
             <geometry>
-                <box size="${camera_length} ${camera_width} ${camera_height}"/>
+                <box size="${camera_length} ${camera_width} ${camera_height}" />
             </geometry>
         </collision>
-        <xacro:box_inertia mass="0.1" lenght="${camera_length}" width="${camera_width}" height="${camera_height}"
-                           xyz="0 0 0" rpy="0 0 0" />
+        <xacro:box_inertia mass="0.1" lenght="${camera_length}" width="${camera_width}"
+            height="${camera_height}"
+            xyz="0 0 0" rpy="0 0 0" />
     </link>
     <joint name="camera_torso_joint" type="fixed">
-        <parent link="torso_link"/>
-        <child link="camera_link"/>
-        <origin xyz="0 ${(torso_width + camera_length) / 2} ${torso_height / 2}" rpy="0 0 ${pi/2}"/>
+        <parent link="torso_link" />
+        <child link="camera_link" />
+        <origin xyz="0 ${(torso_width + camera_length) / 2} ${torso_height / 2}" rpy="0 0 ${pi/2}" />
     </joint>
     <link name="camera_link_optical" />
     <joint name="camera_optical_joint" type="fixed">
-        <origin xyz="0 0 0" rpy="${-pi/2} 0 ${-pi/2}"/>
-        <parent link="camera_link"/>
-        <child link="camera_link_optical"/>
+        <origin xyz="0 0 0" rpy="${-pi/2} 0 ${-pi/2}" />
+        <parent link="camera_link" />
+        <child link="camera_link_optical" />
     </joint>
     <gazebo reference="camera_link">

File: ros2_ws/src/desk_walking_robot_description/urdf/common_properties.xacro (robot description, xacro)
@@ -12,6 +12,6 @@
             <mass value="${mass}" />
             <inertia ixx="${(mass/12) * (width*width + height*height)}" ixy="0" ixz="0"
-                     iyy="${(mass/12) * (lenght*lenght + height*height)}" iyz="0"
-                     izz="${(mass/12) * (lenght*lenght + width*width)}" />
+                iyy="${(mass/12) * (lenght*lenght + height*height)}" iyz="0"
+                izz="${(mass/12) * (lenght*lenght + width*width)}" />
         </inertial>
     </xacro:macro>
@@ -21,6 +21,6 @@
             <mass value="${mass}" />
             <inertia ixx="${(mass/12) * (3*radius*radius + height*height)}" ixy="0" ixz="0"
-                     iyy="${(mass/12) * (3*radius*radius + height*height)}" iyz="0"
-                     izz="${(mass/2) * (radius*radius)}" />
+                iyy="${(mass/12) * (3*radius*radius + height*height)}" iyz="0"
+                izz="${(mass/2) * (radius*radius)}" />
         </inertial>
     </xacro:macro>
@@ -30,6 +30,6 @@
             <mass value="${mass}" />
             <inertia ixx="${(2/5) * mass * radius * radius}" ixy="0" ixz="0"
-                     iyy="${(2/5) * mass * radius * radius}" iyz="0"
-                     izz="${(2/5) * mass * radius * radius}" />
+                iyy="${(2/5) * mass * radius * radius}" iyz="0"
+                izz="${(2/5) * mass * radius * radius}" />
         </inertial>
     </xacro:macro>

File: ros2_ws/src/desk_walking_robot_description/urdf/solid_structure.xacro (robot description, xacro)
@@ -6,5 +6,5 @@
     <xacro:property name="torso_width" value="${0.5 * torso_height}" />
     <xacro:property name="pivot_radius" value="${0.05 * torso_height}" />
-	<xacro:property name="pivot_length" value="${torso_width/8}" />
+    <xacro:property name="pivot_length" value="${torso_width/8}" />
     <xacro:property name="leg_lenght" value="${torso_height / 2}" />
     <xacro:property name="leg_hip_offset" value="${-(leg_lenght / 2)}" />
@@ -12,5 +12,5 @@
     <xacro:property name="foot_height" value="${pivot_radius*1.25}" />
     <xacro:property name="foot_ankle_offset" value="${pivot_radius-(foot_height/2)}" />
-	<!-- for wheels collisions use spheres instead of cylinders -->
+    <!-- for wheels collisions use spheres instead of cylinders -->
     <link name="base_footprint" />
     <link name="torso_link">
@@ -22,5 +22,5 @@
             <material name="blue" />
         </visual>
-		<collision>
+        <collision>
             <geometry>
                 <box size="${torso_length} ${torso_width} ${torso_height}" />
@@ -28,6 +28,6 @@
             <origin xyz="0 0 ${torso_height / 2.0}" rpy="0 0 0" />
         </collision>
-		<xacro:box_inertia mass="5.0" height="${torso_height}" lenght="${torso_length}" width="${torso_width}"
-                           xyz="0 0 ${torso_height / 2.0}" rpy="0 0 0" />
+        <xacro:box_inertia mass="5.0" height="${torso_height}" lenght="${torso_length}"
+            width="${torso_width}" xyz="0 0 ${torso_height / 2.0}" rpy="0 0 0" />
     </link>
     <xacro:macro name="pivot_link" params="prefix xyz rpy">
@@ -54,5 +54,5 @@
             <material name="blue" />
         </visual>
-		<collision>
+        <collision>
             <geometry>
                 <cylinder radius="${torso_length*0.2}" length="${leg_lenght}" />
@@ -60,5 +60,6 @@
             <origin xyz="0 0 ${leg_hip_offset}" rpy="0 0 0" />
         </collision>
-		<xacro:cylinder_inertia mass="2.0" radius="${torso_length*0.2}" height="${leg_lenght}" xyz="0 0 ${leg_hip_offset}" rpy="0 0 0" />
+        <xacro:cylinder_inertia mass="2.0" radius="${torso_length*0.2}" height="${leg_lenght}"
+            xyz="0 0 ${leg_hip_offset}" rpy="0 0 0" />
     </link>
     <link name="left_leg_link">
@@ -70,5 +71,5 @@
             <material name="blue" />
         </visual>
-		<collision>
+        <collision>
             <geometry>
                 <cylinder radius="${torso_length*0.2}" length="${leg_lenght}" />
@@ -76,5 +77,6 @@
             <origin xyz="0 0 ${leg_hip_offset}" rpy="0 0 0" />
         </collision>
-		<xacro:cylinder_inertia mass="2.0" radius="${torso_length*0.2}" height="${leg_lenght}" xyz="0 0 ${leg_hip_offset}" rpy="0 0 0" />
+        <xacro:cylinder_inertia mass="2.0" radius="${torso_length*0.2}" height="${leg_lenght}"
+            xyz="0 0 ${leg_hip_offset}" rpy="0 0 0" />
     </link>
     <link name="right_foot_link">
@@ -86,5 +88,5 @@
             <material name="blue" />
         </visual>
-		<collision>
+        <collision>
             <geometry>
                 <box size="${torso_length*0.5/0.7} ${torso_width*1.1} ${foot_height}" />
@@ -92,6 +94,6 @@
             <origin xyz="0 0 ${foot_ankle_offset}" rpy="0 0 0" />
         </collision>
-		<xacro:box_inertia mass="1.0" lenght="${torso_length*0.5/0.7}" width="${torso_width*1.1}" height="${foot_height}"
-                           xyz="0 0 ${foot_ankle_offset}" rpy="0 0 0" />
+        <xacro:box_inertia mass="1.0" lenght="${torso_length*0.5/0.7}" width="${torso_width*1.1}"
+            height="${foot_height}" xyz="0 0 ${foot_ankle_offset}" rpy="0 0 0" />
     </link>
     <link name="left_foot_link">
@@ -103,5 +105,5 @@
             <material name="blue" />
         </visual>
-		<collision>
+        <collision>
             <geometry>
                 <box size="${torso_length*0.5/0.7} ${torso_width*1.1} ${foot_height}" />
@@ -109,16 +111,16 @@
             <origin xyz="0 0 ${foot_ankle_offset}" rpy="0 0 0" />
         </collision>
-		<xacro:box_inertia mass="1.0" lenght="${torso_length*0.5/0.7}" width="${torso_width*1.1}" height="${foot_height}"
-                           xyz="0 0 ${foot_ankle_offset}" rpy="0 0 0" />
+        <xacro:box_inertia mass="1.0" lenght="${torso_length*0.5/0.7}" width="${torso_width*1.1}"
+            height="${foot_height}" xyz="0 0 ${foot_ankle_offset}" rpy="0 0 0" />
     </link>
     <joint name="base_joint" type="fixed">
         <parent link="base_footprint" />
         <child link="torso_link" />
-        <origin xyz="0 0 ${leg_lenght+foot_height+1.5*pivot_radius}" rpy="0 0 0"/>
+        <origin xyz="0 0 ${leg_lenght+foot_height+1.5*pivot_radius}" rpy="0 0 0" />
     </joint>
     <joint name="right_hip_joint" type="revolute">
         <parent link="torso_link" />
         <child link="right_hip_link" />
-        <origin xyz="${torso_length/2} 0 0" rpy="0 0 0"/>
+        <origin xyz="${torso_length/2} 0 0" rpy="0 0 0" />
         <axis xyz="0 0 1" />
         <limit lower="${-pi/2.0}" upper="${pi/2.0}" velocity="100" effort="100" />
@@ -127,5 +129,5 @@
         <parent link="torso_link" />
         <child link="left_hip_link" />
-        <origin xyz="${-torso_length/2} 0 0" rpy="0 0 0"/>
+        <origin xyz="${-torso_length/2} 0 0" rpy="0 0 0" />
         <axis xyz="0 0 -1" />
         <limit lower="${-pi/2.0}" upper="${pi/2.0}" velocity="100" effort="100" />
@@ -134,15 +136,15 @@
         <parent link="right_hip_link" />
         <child link="right_leg_link" />
-        <origin xyz="0 0 -${pivot_length}" rpy="0 0 0"/>
+        <origin xyz="0 0 -${pivot_length}" rpy="0 0 0" />
     </joint>
     <joint name="left_leg_joint" type="fixed">
         <parent link="left_hip_link" />
         <child link="left_leg_link" />
-        <origin xyz="0 0 -${pivot_length}" rpy="0 0 0"/>
+        <origin xyz="0 0 -${pivot_length}" rpy="0 0 0" />
     </joint>
     <joint name="right_ankle_joint" type="revolute">
         <parent link="right_leg_link" />
         <child link="right_ankle_link" />
-        <origin xyz="0 0 ${leg_ankle_offset}" rpy="0 0 0"/>
+        <origin xyz="0 0 ${leg_ankle_offset}" rpy="0 0 0" />
         <axis xyz="0 1 0" />
         <limit lower="-0.8" upper="0.8" velocity="100" effort="100" />
@@ -151,5 +153,5 @@
         <parent link="left_leg_link" />
         <child link="left_ankle_link" />
-        <origin xyz="0 0 ${leg_ankle_offset}" rpy="0 0 0"/>
+        <origin xyz="0 0 ${leg_ankle_offset}" rpy="0 0 0" />
         <axis xyz="0 -1 0" />
         <limit lower="-0.8" upper="0.8" velocity="100" effort="100" />
@@ -158,10 +160,10 @@
         <parent link="right_ankle_link" />
         <child link="right_foot_link" />
-        <origin xyz="0 0 -${pivot_radius}" rpy="0 0 0"/>
+        <origin xyz="0 0 -${pivot_radius}" rpy="0 0 0" />
     </joint>
     <joint name="left_foot_joint" type="fixed">
         <parent link="left_ankle_link" />
         <child link="left_foot_link" />
-        <origin xyz="0 0 -${pivot_radius}" rpy="0 0 0"/>
+        <origin xyz="0 0 -${pivot_radius}" rpy="0 0 0" />
     </joint>
 </robot>
