Commit message: added limits to rotation/revolute and use pi for math

File: ros2_ws/src/desk_walking_robot_description/urdf/solid_structure.xacro (robot description, xacro)
@@ -31,8 +31,8 @@
         </link>
     </xacro:macro>
-    <xacro:pivot_link prefix="right_hip" rpy="0 1.57 0" />
-    <xacro:pivot_link prefix="left_hip" rpy="0 1.57 0" />
-    <xacro:pivot_link prefix="right_ankle" rpy="1.57 0 0" />
-    <xacro:pivot_link prefix="left_ankle" rpy="1.57 0 0" />
+    <xacro:pivot_link prefix="right_hip" rpy="0 ${pi/2.0} 0" />
+    <xacro:pivot_link prefix="left_hip" rpy="0 ${pi/2.0} 0" />
+    <xacro:pivot_link prefix="right_ankle" rpy="${pi/2.0} 0 0" />
+    <xacro:pivot_link prefix="left_ankle" rpy="${pi/2.0} 0 0" />
     <link name="right_leg_link">
         <visual>
@@ -76,15 +76,17 @@
         <origin xyz="0 0 ${leg_lenght+foot_height+1.5*pivot_radius}" rpy="0 0 0"/>
     </joint>
-    <joint name="right_hip_joint" type="continuous">
+    <joint name="right_hip_joint" type="revolute">
         <parent link="base_link" />
         <child link="right_hip_link" />
         <origin xyz="${torso_length/2} 0 0" rpy="0 0 0"/>
         <axis xyz="-1 0 0" />
+        <limit lower="${-pi/2.0}" upper="${pi/2.0}" velocity="100" effort="100" />
     </joint>
-    <joint name="left_hip_joint" type="continuous">
+    <joint name="left_hip_joint" type="revolute">
         <parent link="base_link" />
         <child link="left_hip_link" />
         <origin xyz="${-torso_length/2} 0 0" rpy="0 0 0"/>
         <axis xyz="-1 0 0" />
+        <limit lower="${-pi/2.0}" upper="${pi/2.0}" velocity="100" effort="100" />
     </joint>
     <joint name="right_leg_joint" type="fixed">
@@ -98,15 +100,17 @@
         <origin xyz="0 0 -${pivot_radius}" rpy="0 0 0"/>
     </joint>
-    <joint name="right_ankle_joint" type="continuous">
+    <joint name="right_ankle_joint" type="revolute">
         <parent link="right_leg_link" />
         <child link="right_ankle_link" />
         <origin xyz="0 0 ${leg_ankle_offset}" rpy="0 0 0"/>
         <axis xyz="0 1 0" />
+        <limit lower="-0.8" upper="0.8" velocity="100" effort="100" />
     </joint>
-    <joint name="left_ankle_joint" type="continuous">
+    <joint name="left_ankle_joint" type="revolute">
         <parent link="left_leg_link" />
         <child link="left_ankle_link" />
         <origin xyz="0 0 ${leg_ankle_offset}" rpy="0 0 0"/>
         <axis xyz="0 -1 0" />
+        <limit lower="-0.8" upper="0.8" velocity="100" effort="100" />
     </joint>
     <joint name="right_foot_joint" type="fixed">

Commit message: my_desk_robot gazebo changes. Sim is moving in Gazebo

File: ros2_ws/src/desk_walking_robot_description/urdf/solid_structure.xacro (robot description, xacro)
@@ -2,5 +2,5 @@
 <!-- Xacro allows to use macros and properties to generate URDF files -->
 <robot xmlns:xacro="http://www.ros.org/wiki/xacro">
-    <xacro:property name="torso_height" value="1" />
+    <xacro:property name="torso_height" value="0.4" />
     <xacro:property name="torso_length" value="${0.7 * torso_height}" />
     <xacro:property name="torso_width" value="${0.5 * torso_height}" />
@@ -28,5 +28,5 @@
             <origin xyz="0 0 ${torso_height / 2.0}" rpy="0 0 0" />
         </collision>
-        <xacro:box_inertia mass="5.0" height="${torso_height}" lenght="${torso_length}"
+        <xacro:box_inertia mass="2.0" height="${torso_height}" lenght="${torso_length}"
             width="${torso_width}" xyz="0 0 ${torso_height / 2.0}" rpy="0 0 0" />
     </link>
@@ -60,5 +60,5 @@
             <origin xyz="0 0 ${leg_hip_offset}" rpy="0 0 0" />
         </collision>
-        <xacro:cylinder_inertia mass="2.0" radius="${torso_length*0.2}" height="${leg_lenght}"
+        <xacro:cylinder_inertia mass="1.0" radius="${torso_length*0.2}" height="${leg_lenght}"
             xyz="0 0 ${leg_hip_offset}" rpy="0 0 0" />
     </link>
@@ -77,5 +77,5 @@
             <origin xyz="0 0 ${leg_hip_offset}" rpy="0 0 0" />
         </collision>
-        <xacro:cylinder_inertia mass="2.0" radius="${torso_length*0.2}" height="${leg_lenght}"
+        <xacro:cylinder_inertia mass="1.0" radius="${torso_length*0.2}" height="${leg_lenght}"
             xyz="0 0 ${leg_hip_offset}" rpy="0 0 0" />
     </link>
@@ -83,5 +83,5 @@
         <visual>
             <geometry>
-                <box size="${torso_length*0.5/0.7} ${torso_width*1.1} ${foot_height}" />
+                <box size="${torso_length*0.5/0.6} ${torso_width*1.3} ${foot_height}" />
             </geometry>
             <origin xyz="0 0 ${foot_ankle_offset}" rpy="0 0 0" />
@@ -90,5 +90,5 @@
         <collision>
             <geometry>
-                <box size="${torso_length*0.5/0.7} ${torso_width*1.1} ${foot_height}" />
+                <box size="${torso_length*0.5/0.6} ${torso_width*1.3} ${foot_height}" />
             </geometry>
             <origin xyz="0 0 ${foot_ankle_offset}" rpy="0 0 0" />
@@ -100,5 +100,5 @@
         <visual>
             <geometry>
-                <box size="${torso_length*0.5/0.7} ${torso_width*1.1} ${foot_height}" />
+                <box size="${torso_length*0.5/0.6} ${torso_width*1.3} ${foot_height}" />
             </geometry>
             <origin xyz="0 0 ${foot_ankle_offset}" rpy="0 0 0" />
@@ -107,5 +107,5 @@
         <collision>
             <geometry>
-                <box size="${torso_length*0.5/0.7} ${torso_width*1.1} ${foot_height}" />
+                <box size="${torso_length*0.5/0.6} ${torso_width*1.3} ${foot_height}" />
             </geometry>
             <origin xyz="0 0 ${foot_ankle_offset}" rpy="0 0 0" />
@@ -125,4 +125,5 @@
         <axis xyz="0 0 1" />
         <limit lower="${-pi/2.0}" upper="${pi/2.0}" velocity="100" effort="100" />
+        <dynamics damping="0.5" friction="0.3" />
     </joint>
     <joint name="left_hip_joint" type="revolute">
@@ -132,4 +133,5 @@
         <axis xyz="0 0 -1" />
         <limit lower="${-pi/2.0}" upper="${pi/2.0}" velocity="100" effort="100" />
+        <dynamics damping="0.5" friction="0.3" />
     </joint>
     <joint name="right_leg_joint" type="fixed">
@@ -149,4 +151,5 @@
         <axis xyz="0 1 0" />
         <limit lower="-0.8" upper="0.8" velocity="100" effort="100" />
+        <dynamics damping="0.5" friction="0.3" />
     </joint>
     <joint name="left_ankle_joint" type="revolute">
@@ -156,4 +159,5 @@
         <axis xyz="0 -1 0" />
         <limit lower="-0.8" upper="0.8" velocity="100" effort="100" />
+        <dynamics damping="0.5" friction="0.3" />
     </joint>
     <joint name="right_foot_joint" type="fixed">

File: ros2_ws/src/desk_walking_robot_description/urdf/solid_structure_gazebo.xacro (robot description, xacro)
@@ -29,4 +29,5 @@
             name="gz::sim::systems::JointPositionController">
             <joint_name>right_hip_joint</joint_name>
+            <p_gain>15.0</p_gain>
         </plugin>
     </gazebo>
@@ -36,4 +37,5 @@
             name="gz::sim::systems::JointPositionController">
             <joint_name>left_hip_joint</joint_name>
+            <p_gain>15.0</p_gain>
         </plugin>
     </gazebo>
@@ -43,4 +45,5 @@
             name="gz::sim::systems::JointPositionController">
             <joint_name>right_ankle_joint</joint_name>
+            <p_gain>15.0</p_gain>
         </plugin>
     </gazebo>
@@ -50,4 +53,5 @@
             name="gz::sim::systems::JointPositionController">
             <joint_name>left_ankle_joint</joint_name>
+            <p_gain>15.0</p_gain>
         </plugin>
     </gazebo>
