Commit message: Gazebo project finished

File: ros2_ws/src/my_robot_description/urdf/arm.xacro (robot description, xacro)
@@ -21,5 +21,5 @@
             <origin xyz="0 0 0" rpy="0 0 0" />
         </collision>
-        <xacro:box_inertia m="5.0" x="${arm_base_length}" y="${arm_base_width}" z="${arm_base_height}"
+        <xacro:box_inertia m="0.5" x="${arm_base_length}" y="${arm_base_width}" z="${arm_base_height}"
                            o_xyz="0 0 0" o_rpy="0 0 0" />
     </link>

File: ros2_ws/src/my_robot_description/urdf/my_robot.urdf.xacro (robot description, xacro)
@@ -7,3 +7,8 @@
     <xacro:include filename="arm.xacro" />
     <xacro:include filename="arm_gazebo.xacro" />
+    <joint name="base_to_arm" type="fixed">
+        <origin xyz="0 0 ${base_height}" rpy="0 0 ${pi/2}"/>
+        <parent link="base_link"/>
+        <child link="arm_footprint"/>
+    </joint>
 </robot>
